File: IRF510-Amplifier.kicad_pcb (KiCad board)
At the start: 2 copper layers, 144.8 x 72.8 mm, 39 parts, among them J1 Jack-DC, J2 BNC, J3 BNC, Q1 2N3904-SMD, Q2 2SC5706, Q4 IRF540N, T1 T37-6 15T:7T, U6 MCP1703A-2502_SOT223

Commit message: Update IRF510-Amplifier.kicad_pcb
Parts:
- moved   0.74 mm to (159.0, 64.5)
Routing:
- net Net-(C2-Pad2): track 34.5 -> 33.4 mm
- removed copper zone on B.Cu, net GND
- removed copper zone on F.Cu, net GND
Changed lines of the file:
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@@
     (mod_text_size 1 1)
     (mod_text_width 0.15)
-    (pad_size 1.778 1.778)
-    (pad_drill 0.8)
+    (pad_size 5 5)
+    (pad_drill 2.7)
     (pad_to_mask_clearance 0.051)
     (solder_mask_min_width 0.25)
@@
     (add_net "Net-(D1-Pad2)")
     (add_net "Net-(Q2-Pad3)")
-    (add_net "Net-(RV1-Pad1)")
   )
   (module MountingHole:MountingHole_2.5mm_Pad (layer F.Cu)
@@
     (fp_circle (center 0 0) (end 2.5 0) (layer Cmts.User) (width 0.15))
     (fp_circle (center 0 0) (end 2.75 0) (layer F.CrtYd) (width 0.05))
-    (pad 1 thru_hole circle (at 0 0) (size 5 5) (drill 2.5) (layers *.Cu *.Mask))
+    (pad 1 thru_hole circle (at 0 0) (size 5 5) (drill 2.7) (layers *.Cu *.Mask))
   )
   (module MountingHole:MountingHole_2.5mm_Pad (layer F.Cu)
-    (at 159 65.24)
+    (at 159 64.5)
     (descr "Mounting Hole 2.5mm")
     (tags "mounting hole 2.5mm")
@@
       (effects (font (size 1 1) (thickness 0.15)))
     )
-    (pad 1 thru_hole circle (at 0 0) (size 5 5) (drill 2.5) (layers *.Cu *.Mask))
+    (pad 1 thru_hole circle (at 0 0) (size 5 5) (drill 2.7) (layers *.Cu *.Mask))
   )
   (module Package_TO_SOT_SMD:TO-252-3_TabPin2 (layer F.Cu)
@@
   (segment (start 142.58 82.34) (end 145.4 85.16) (width 1) (layer F.Cu) (net 16))
   (segment (start 140.1375 82.34) (end 142.58 82.34) (width 1) (layer F.Cu) (net 16))
-  (segment (start 163 82.2325) (end 163 80.28) (width 1) (layer F.Cu) (net 16))
-  (segment (start 160.0725 85.16) (end 163 82.2325) (width 1) (layer F.Cu) (net 16))
-  (segment (start 145.4 85.16) (end 160.0725 85.16) (width 1) (layer F.Cu) (net 16))
+  (segment (start 163 80.28) (end 155.28 80.28) (width 1) (layer F.Cu) (net 16))
+  (segment (start 150.4 85.16) (end 145.4 85.16) (width 1) (layer F.Cu) (net 16))
+  (segment (start 155.28 80.28) (end 150.4 85.16) (width 1) (layer F.Cu) (net 16))
   (segment (start 140.1375 79.765) (end 140.1375 76.7) (width 1) (layer F.Cu) (net 17))
   (segment (start 138.2625 81.64) (end 140.1375 79.765) (width 1) (layer F.Cu) (net 17))
@@
   (segment (start 150.125 75) (end 150.4 74.725) (width 1) (layer F.Cu) (net 19))
   (segment (start 145.4 75) (end 150.125 75) (width 1) (layer F.Cu) (net 19))
-  (zone (net 1) (net_name GND) (layer F.Cu) (hatch edge 0.508)
-    (connect_pads (clearance 0.508))
-    (min_thickness 0.254)
-    (fill yes (arc_segments 32) (thermal_gap 0.508) (thermal_bridge_width 0.508))
-    (polygon
-      (pts
-        (xy 220.4 102.6) (xy 75.2 102.6) (xy 75.2 29.8) (xy 220.4 29.8)
-      )
-    )
-  )
-  (zone (net 1) (net_name GND) (layer B.Cu) (hatch edge 0.508)
-    (connect_pads (clearance 0.508))
-    (min_thickness 0.254)
-    (fill yes (arc_segments 32) (thermal_gap 0.508) (thermal_bridge_width 0.508))
-    (polygon
-      (pts
-        (xy 220 102.6) (xy 75.4 102.6) (xy 75.4 30) (xy 220 30)
-      )
-    )
-  )
 )

Commit message: l
Parts:
- Q4: value IRF540N -> IRF510
Routing:
- added copper zone on B.Cu, net GND
- added copper zone on F.Cu, net GND

Commit message: reorg
Parts:
- removed the   at (159.0, 90.2)
- removed the   at (159.0, 64.5)
- added  : , MountingHole:MountingHole_3.2mm_M3, F.Cu at (79.2, 97.8)
- added  : , MountingHole:MountingHole_3.2mm_M3, F.Cu at (198.4, 97.8)
- added  : , MountingHole:MountingHole_3.2mm_M3, F.Cu at (198.6, 23.2)
- added  : , MountingHole:MountingHole_3.2mm_M3, F.Cu at (79.2, 23.4)
- added  : , Xenir:Heatsink_Mounting_25mm, F.Cu at (159.6, 64.8)
- added C6: .1uF, Xenir:Capacitor 0805, F.Cu at (82.6, 65.0)
- added J4: Audio_Jack, Xenir:Audio_Jack, B.Cu at (81.2, 58.2)
- added Q3: BS170F, Package_TO_SOT_SMD:SOT-23, F.Cu at (84.4, 65.0)
- added Q5: IRFU9024, Package_TO_SOT_THT:TO-251-3_Vertical, F.Cu at (89.0, 60.4)
- added R3: 10k, Xenir:Resistor 0805, F.Cu at (77.5, 60.7)
- added R4: 10k, Xenir:Resistor 0805, F.Cu at (95.8, 65.0)
- added R5: 1.5k, Xenir:Resistor 0805, F.Cu at (84.1, 62.5)
- added R7: 10k, Xenir:Resistor 0805, F.Cu at (91.8, 65.0)
- moved C57 23.6 mm to (173.1, 53.9), turned to 0 degrees
- moved C3 20.2 mm to (178.4, 63.4), turned to 0 degrees
- moved C8 19.1 mm to (183.6, 83.0), turned to 180 degrees
- moved J2 18.6 mm to (194.8, 81.0)
- moved L3 16.0 mm to (188.0, 60.2), turned to 270 degrees
- moved J1 10.2 mm to (89.4, 38.0)
- moved C5 9.53 mm to (183.6, 70.6), turned to 180 degrees
- moved C7 5.14 mm to (187.2, 73.2), turned to 90 degrees
- moved L4 4.60 mm to (188.0, 73.6), turned to 270 degrees
- moved J3 1.63 mm to (82.8, 81.2)
Connections:
- U6 pad 1: +12V -> Net-(Q5-Pad2)
Routing:
- net Net-(J4-PadRING): track 0.00 -> 20.1 mm
- net +12V: track 123.6 -> 142.3 mm, vias 0 -> 1
- net Net-(Q5-Pad2): track 0.00 -> 13.8 mm
- net Net-(Q5-Pad1): track 0.00 -> 8.55 mm
- net Net-(C6-Pad1): track 0.00 -> 8.06 mm
- net Net-(C7-Pad1): track 21.3 -> 15.3 mm
- net Net-(Q3-Pad3): track 0.00 -> 4.25 mm
- net Net-(C57-Pad1): track 38.2 -> 33.9 mm
- net Net-(C3-Pad1): track 16.0 -> 12.5 mm
Other:
- board size 144.8 x 72.8 mm -> 126.4 x 81.6 mm
- board text added: "10W Amplifier"
