File: IRF510-Amplifier.kicad_pcb (KiCad board)
At the start: 2 copper layers, 126.4 x 81.6 mm, 50 parts, among them J1 Jack-DC, J2 BNC, J3 BNC, J4 Audio_Jack, Q1 2N3904-SMD, Q2 2SC5706, Q3 BS170F, Q4 IRF510, Q5 IRFU9024, T1 T37-6 15T:7T, U6 MCP1703A-2502_SOT223

Commit message: updates after 1st test
Parts:
- added C10: .1uF, Xenir:Capacitor 0805, F.Cu at (150.1, 91.1)
- added R8: 1k, Xenir:Resistor 0805, F.Cu at (136.9, 54.7)
- added R9: 2.7k, Xenir:Resistor 0805, F.Cu at (150.1, 87.4)
- R55: value 10 -> 5.1
- T1: value T37-6 15T:7T -> T37-43 8T:4T
- moved C11 11.8 mm to (93.2, 35.4), turned to 90 degrees
Connections:
- C53 pad 1: +12V -> 12V-On
- Q5 pad 2: Net-(Q5-Pad2) -> 12V-On
- RV2 pad 2: Net-(C2-Pad2) -> Net-(R9-Pad1)
- T1 pad C1B: +12V -> 12V-On
- U6 pad 1: Net-(Q5-Pad2) -> 12V-On
Routing:
- net 12V-On: track 0.00 -> 70.4 mm
- net +12V: track 142.3 -> 110.6 mm
- net Net-(Q5-Pad2): track 13.8 -> 0.00 mm
- net Net-(R9-Pad1): track 0.00 -> 7.83 mm
- net GND: track 21.0 -> 15.5 mm
- net +5V: track 88.2 -> 93.2 mm
- net Net-(C1-Pad1): track 4.47 -> 8.38 mm
- net Net-(C2-Pad2): track 33.4 -> 31.3 mm
