File: IRF510-Amplifier.sch (KiCad schematic (older format))
At the start: 37 parts, among them J1 Jack-DC, J2 BNC, J3 BNC, Q1 2N3904-SMD, Q2 2SC5706, Q4 IRF540N, T1 T37-6 15T:7T, U6 MCP1703A-2502_SOT223

Commit message: l
Parts:
- Q4: value IRF540N -> IRF510
Changed lines of the file:
@@
 P 6850 2950
 F 0 "Q4" H 7100 3025 50  0000 L CNN
-F 1 "IRF540N" H 7100 2950 50  0000 L CNN
+F 1 "IRF510" H 7100 2950 50  0000 L CNN
 F 2 "Package_TO_SOT_THT:TO-220-3_Vertical" H 7100 2875 50  0001 L CIN
 F 3 "http://www.irf.com/product-info/datasheets/data/irf540n.pdf" H 6850 2950 50  0001 L CNN

Commit message: reorg
Parts:
- added C6: .1uF, Xenir:Capacitor 0805, symbol Xenir:Capacitor
- added J4: Audio_Jack, Xenir:Audio_Jack, symbol Xenir:Audio_Jack
- added Q3: BS170F, Package_TO_SOT_SMD:SOT-23, symbol Transistor_FET:BS170F
- added Q5: IRFU9024, Package_TO_SOT_THT:TO-251-3_Vertical, symbol Xenir:IRFU9024
- added R3, R4, R7: 10k, Xenir:Resistor 0805, symbol Xenir:Resistor
- added R5: 1.5k, Xenir:Resistor 0805, symbol Xenir:Resistor
Connections:
- net +12V: now also Q5.3 (S), R4.1; no longer U6.1 (VI)
- net GND: now also C6.2, J4.SLEEVE, Q3.2 (S), R3.1
- new net: Q5.2 (D), U6.1 (VI)
- new net: Q5.1 (G), R4.2, R7.1
- new net: Q3.3 (D), R7.2
- new net: C6.1, Q3.1 (G), R5.1
- new net: J4.RING, J4.RSH, J4.TIP, J4.TSH, R3.2, R5.2
Other:
- moved on the sheet: C11, C14, J1, U6

Commit message: updates after 1st test
Parts:
- added C10: .1uF, Xenir:Capacitor 0805, symbol Xenir:Capacitor
- added R8: 1k, Xenir:Resistor 0805, symbol Xenir:Resistor
- added R9: 2.7k, Xenir:Resistor 0805, symbol Xenir:Resistor
- R55: value 10 -> 5.1
- T1: value T37-6 15T:7T -> T37-43 8T:4T
Connections:
- net +12V: no longer C53.1, T1.C1B
- net +5V: now also C10.1
- net GND: now also C10.2, R8.2
- net 12V-On: now reaches Q5.2 (D), U6.1 (VI)
- net 12V-On: now also C53.1, T1.C1B
- net at C2.2, D1.1 (K), Q4.1 (G): now also R9.2; no longer RV2.2
- net at C1.1, T1.C2B: now also R8.1
- new net: R9.1, RV2.2
Other:
- moved on the sheet: RV2
Changed lines of the file:
@@
 P 4000 4550
 F 0 "R55" H 4000 4625 28  0000 C CNN
-F 1 "10" H 4000 4475 28  0000 C CNN
+F 1 "5.1" H 4000 4475 28  0000 C CNN
 F 2 "Xenir:Resistor 0805" H 4000 4450 50  0001 C CNN
 F 3 "" H 4000 4450 50  0001 C CNN
@@
 	4000 3650 4000 3900
 Connection ~ 4000 3650
-$Comp
-L power:+12V #PWR0106
-U 1 1 5F4CAB18
-P 4000 2600
-F 0 "#PWR0106" H 4000 2450 50  0001 C CNN
-F 1 "+12V" H 4000 2740 50  0000 C CNN
-F 2 "" H 4000 2600 50  0001 C CNN
-F 3 "" H 4000 2600 50  0001 C CNN
-	1    4000 2600
-	-1   0    0    -1
-$EndComp
 $Comp
 L Xenir:Capacitor C53
@@
 $EndComp
 Wire Wire Line
-	4000 2600 4000 2750
+	8300 4250 8300 4400
 Wire Wire Line
 	3700 2750 3700 2900
@@
 P 4400 2600
 F 0 "T1" H 4400 1750 50  0000 C CNN
-F 1 "T37-6 15T:7T " H 4400 2600 50  0000 C CNN
+F 1 "T37-43 8T:4T" H 4400 2600 50  0000 C CNN
 F 2 "Xenir:T37 Transformer" H 4400 2600 50  0001 C CNN
 F 3 "" H 4400 2600 50  0001 C CNN
@@
 $EndComp
 Connection ~ 4000 3350
-Connection ~ 4000 2750
 $Comp
 L Device:R_POT RV1
@@
 $EndComp
 Wire Wire Line
-	4800 2750 5000 2750
+	4800 2750 4900 2750
 Wire Wire Line
 	5300 2750 5450 2750
@@
 L Device:R_POT RV2
 U 1 1 61016758
-P 6350 2400
-F 0 "RV2" V 6175 2400 50  0000 C CNN
-F 1 "R_POT" V 6250 2400 50  0000 C CNN
-F 2 "Xenir:Trimpot Vertical" H 6350 2400 50  0001 C CNN
-F 3 "~" H 6350 2400 50  0001 C CNN
-	1    6350 2400
+P 6350 2050
+F 0 "RV2" V 6175 2050 50  0000 C CNN
+F 1 "R_POT" V 6250 2050 50  0000 C CNN
+F 2 "Xenir:Trimpot Vertical" H 6350 2050 50  0001 C CNN
+F 3 "~" H 6350 2050 50  0001 C CNN
+	1    6350 2050
 	0    1    1    0
 $EndComp
@@
 L power:GND #PWR0112
 U 1 1 61016E3B
-P 6600 2550
-F 0 "#PWR0112" H 6600 2300 50  0001 C CNN
-F 1 "GND" H 6600 2400 50  0000 C CNN
-F 2 "" H 6600 2550 50  0001 C CNN
-F 3 "" H 6600 2550 50  0001 C CNN
-	1    6600 2550
-	1    0    0    -1
-$EndComp
-Wire Wire Line
-	6600 2550 6600 2400
-Wire Wire Line
-	6600 2400 6500 2400
+P 6600 2200
+F 0 "#PWR0112" H 6600 1950 50  0001 C CNN
+F 1 "GND" H 6600 2050 50  0000 C CNN
+F 2 "" H 6600 2200 50  0001 C CNN
+F 3 "" H 6600 2200 50  0001 C CNN
+	1    6600 2200
+	1    0    0    -1
+$EndComp
+Wire Wire Line
+	6600 2200 6600 2050
+Wire Wire Line
+	6600 2050 6500 2050
 $Comp
 L power:+5V #PWR0113
 U 1 1 61018572
-P 6050 2300
-F 0 "#PWR0113" H 6050 2150 50  0001 C CNN
-F 1 "+5V" H 6050 2440 50  0000 C CNN
-F 2 "" H 6050 2300 50  0001 C CNN
-F 3 "" H 6050 2300 50  0001 C CNN
-	1    6050 2300
-	1    0    0    -1
-$EndComp
-Wire Wire Line
-	6200 2400 6050 2400
-Wire Wire Line
-	6050 2400 6050 2300
+P 6050 1950
+F 0 "#PWR0113" H 6050 1800 50  0001 C CNN
+F 1 "+5V" H 6050 2090 50  0000 C CNN
+F 2 "" H 6050 1950 50  0001 C CNN
+F 3 "" H 6050 1950 50  0001 C CNN
+	1    6050 1950
+	1    0    0    -1
+$EndComp
+Wire Wire Line
+	6200 2050 6050 2050
+Wire Wire Line
+	6050 2050 6050 1950
 Wire Wire Line
 	6650 2950 6350 2950
-Wire Wire Line
-	6350 2950 6350 2550
 $Comp
 L power:+12V #PWR0114
@@
 	1    0    0    -1
 $EndComp
-Wire Wire Line
-	8100 4400 8550 4400
 Connection ~ 7100 4400
 $Comp
@@
 Connection ~ 6400 5600
 Connection ~ 7200 5600
+Text GLabel 8300 4250 1    50   Input ~ 0
+12V-On
+Wire Wire Line
+	8100 4400 8300 4400
+Connection ~ 8300 4400
+Wire Wire Line
+	8300 4400 8550 4400
+Wire Wire Line
+	4000 2600 4000 2750
+Text GLabel 4000 2600 1    50   Input ~ 0
+12V-On
+Connection ~ 4000 2750
+$Comp
+L Xenir:Resistor R8
+U 1 1 60F5B137
+P 4900 2950
+F 0 "R8" H 4900 3025 28  0000 C CNN
+F 1 "1k" H 4900 2875 28  0000 C CNN
+F 2 "Xenir:Resistor 0805" H 4900 2850 50  0001 C CNN
+F 3 "" H 4900 2850 50  0001 C CNN
+	1    4900 2950
+	0    1    1    0
+$EndComp
+Connection ~ 4900 2750
+Wire Wire Line
+	4900 2750 5000 2750
+$Comp
+L power:GND #PWR0106
+U 1 1 60F5C617
+P 4900 3150
+F 0 "#PWR0106" H 4900 2900 50  0001 C CNN
+F 1 "GND" H 4900 3000 50  0000 C CNN
+F 2 "" H 4900 3150 50  0001 C CNN
+F 3 "" H 4900 3150 50  0001 C CNN
+	1    4900 3150
+	1    0    0    -1
+$EndComp
+$Comp
+L Xenir:Resistor R9
+U 1 1 60F799F0
+P 6350 2500
+F 0 "R9" H 6350 2575 28  0000 C CNN
+F 1 "2.7k" H 6350 2425 28  0000 C CNN
+F 2 "Xenir:Resistor 0805" H 6350 2400 50  0001 C CNN
+F 3 "" H 6350 2400 50  0001 C CNN
+	1    6350 2500
+	0    1    1    0
+$EndComp
+Wire Wire Line
+	6350 2200 6350 2300
+Wire Wire Line
+	6350 2700 6350 2950
+$Comp
+L Xenir:Capacitor C10
+U 1 1 60F7F48C
+P 6050 2200
+F 0 "C10" H 6050 2325 28  0000 C CNN
+F 1 ".1uF" H 6050 2075 28  0000 C CNN
+F 2 "Xenir:Capacitor 0805" H 6050 2050 50  0001 C CNN
+F 3 "" H 6050 2050 50  0001 C CNN
+	1    6050 2200
+	0    1    1    0
+$EndComp
+Connection ~ 6050 2050
+$Comp
+L power:GND #PWR0126
+U 1 1 60F801C5
+P 6050 2350
+F 0 "#PWR0126" H 6050 2100 50  0001 C CNN
+F 1 "GND" H 6050 2200 50  0000 C CNN
+F 2 "" H 6050 2350 50  0001 C CNN
+F 3 "" H 6050 2350 50  0001 C CNN
+	1    6050 2350
+	1    0    0    -1
+$EndComp
 $EndSCHEMATC
